Commit message: tut 4.1

File: install/diff_drive_robot_gz_sim/share/diff_drive_robot_gz_sim/urdf/ICTE4001_MRobot_sensor.urdf.xacro (robot description, xacro)
@@ -67,7 +67,4 @@
         <xacro:box_inertia m="15.0" w="${base_width}" d="${base_length}" h="${base_height}"/>
     </link>
-    <gazebo reference="base_link">
-        <material>Gazebo/Red</material>
-    </gazebo>
     <joint name="base_joint" type="fixed">
         <parent link="base_footprint"/>
@@ -112,5 +109,4 @@
             <minDepth>0.0001</minDepth>
             <maxVel>1.0</maxVel>
-            <material>Gazebo/DarkGrey</material>
 		</gazebo>
         <ros2_control name="${prefix}_link_controller" type="system">
@@ -151,5 +147,4 @@
 		<mu1>0.01</mu1>
 		<mu2>0.01</mu2>
-		<material>Gazebo/White</material>
 	</gazebo>
     <joint name="caster_joint" type="fixed">
